Commit message: Cosmetics: added some visual elements to the rocket

File: modelrocket.urdf (robot description, URDF)
Before this commit: robot rocket, 1 links, 0 joints
Links:
- added link booster_link, mass 0.001; collision cylinder length=0.5 radius=0.25; visual cylinder length=0.5 radius=0.25
- added link leg_1, mass 0.00; collision box size=0.05 0.7 0.05; visual box size=0.05 0.7 0.05
- added link leg_2, mass 0.00; collision box size=0.05 0.7 0.05; visual box size=0.05 0.7 0.05
- added link leg_3, mass 0.00; collision box size=0.05 0.7 0.05; visual box size=0.05 0.7 0.05
- added link top_hat_link, mass 0.001; collision cylinder length=0.3 radius=0.13; visual cylinder length=0.3 radius=0.13
- added link top_link, mass 0.001; collision cylinder length=0.5 radius=0.25; visual cylinder length=0.5 radius=0.25
Joints:
- added joint booster_joint: type fixed, parent base_link, child booster_link, origin xyz=0 0 -2 rpy=0 0 0
- added joint leg_1_joint: type fixed, parent base_link, child leg_1, origin xyz=0.0 0.35 -2.4 rpy=0 0 0
- added joint leg_2_joint: type fixed, parent base_link, child leg_2, origin xyz=0.3031 -0.175 -2.4 rpy=0 0 4.188
- added joint leg_3_joint: type fixed, parent base_link, child leg_3, origin xyz=-0.3031 -0.175 -2.4 rpy=0 0 -4.188
- added joint top_hat_joint: type fixed, parent base_link, child top_hat_link, origin xyz=0 0 2.8 rpy=0 0 0
- added joint top_joint: type fixed, parent base_link, child top_link, origin xyz=0 0 2.5 rpy=0 0 0

Commit message: WIP: landing gear

File: modelrocket.urdf (robot description, URDF)
Before this commit: robot rocket, 7 links, 6 joints
Links:
- link leg_1: mass 0.00 -> 0.01
- link leg_2: mass 0.00 -> 0.01
- link leg_3: mass 0.00 -> 0.01
Joints:
- joint leg_1_joint: axis (none) -> 1 0 0; limit (none) -> lower=-1.6 upper=1.6 effort=1000.0 velocity=1.0; type fixed -> revolute
- joint leg_2_joint: axis (none) -> -0.175 -0.3031 0; limit (none) -> lower=-1.6 upper=1.6 effort=1000.0 velocity=1.0; type fixed -> revolute
- joint leg_3_joint: axis (none) -> -0.175 0.3031 0; limit (none) -> lower=-1.6 upper=1.6 effort=1000.0 velocity=1.0; type fixed -> revolute

Commit message: Removed WIP landing gear for now

File: modelrocket.urdf (robot description, URDF)
Before this commit: robot rocket, 7 links, 6 joints
Links:
- link leg_1: mass 0.01 -> 0.00
- link leg_2: mass 0.01 -> 0.00
- link leg_3: mass 0.01 -> 0.00
Joints:
- joint leg_1_joint: axis 1 0 0 -> (none); limit lower=-1.6 upper=1.6 effort=1000.0 velocity=1.0 -> (none); type revolute -> fixed
- joint leg_2_joint: axis -0.175 -0.3031 0 -> (none); limit lower=-1.6 upper=1.6 effort=1000.0 velocity=1.0 -> (none); type revolute -> fixed
- joint leg_3_joint: axis -0.175 0.3031 0 -> (none); limit lower=-1.6 upper=1.6 effort=1000.0 velocity=1.0 -> (none); type revolute -> fixed
